File: RicardoBlackBox.kicad_pcb (KiCad board)
At the start: 2 copper layers, 62 parts, among them J1 RBUS, J3 USB_C_Receptacle_USB2.0, U1 ESP32-S3, U4 SN65HVD230, U5 LTC4411, U6 SC4216H, U7 LTC4411, Y1 40MHz±10ppm

Commit message: 4th
Parts:
- moved H3 95.7 mm to (57.6, 113.9)
- moved H4 75.6 mm to (98.2, 115.7)
- moved H2 69.7 mm to (57.3, 76.9)
- moved D12 68.1 mm to (102.1, 100.0), turned to 180 degrees
- moved C36 67.8 mm to (98.6, 98.6), turned to 180 degrees
- moved C35 63.6 mm to (99.2, 100.0)
- moved C37 63.3 mm to (98.5, 101.5), turned to 180 degrees
- moved R29 61.9 mm to (96.6, 99.6)
- moved C34 61.9 mm to (86.5, 100.5)
- moved R30 60.8 mm to (96.6, 101.1)
- moved TP19 59.0 mm to (63.8, 84.2)
- moved C33 57.9 mm to (86.8, 102.2)
- moved U4 56.2 mm to (91.9, 100.4)
- moved TP18 56.1 mm to (58.2, 84.3)
- moved TP17 55.0 mm to (58.2, 82.1)
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Routing:
- net +3V3: track 0.00 -> 16.8 mm
- net GND: track 0.00 -> 13.3 mm
- net /CAN+: track 0.00 -> 10.4 mm
- net /CAN-: track 0.00 -> 10.1 mm
- net Net-(C25-Pad2): track 0.00 -> 8.12 mm
- net /Data-: track 0.00 -> 8.01 mm
- net /Data+: track 0.00 -> 5.85 mm
- net VBUS: track 0.00 -> 5.69 mm
- net Net-(C35-Pad1): track 0.00 -> 5.02 mm
- net Net-(C14-Pad1): track 0.00 -> 3.68 mm
- net /CHIP_PU: track 0.00 -> 3.48 mm
- net /BOOT: track 0.00 -> 2.60 mm
- net Net-(R24-Pad2): track 0.00 -> 1.78 mm
- net Net-(R28-Pad1): track 0.00 -> 1.77 mm
- net Net-(C13-Pad1): track 0.00 -> 1.45 mm
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