File: RicardoBlackBox.kicad_sch (KiCad schematic)
At the start: 42 parts, among them J1 RBUS, U1 ESP32-S3, U5 LTC4411, Y1 40MHz±10ppm

Commit message: PushingSecondSchematic
Parts:
- removed J?: USB_C_Receptacle_USB2.0, Connector_USB:USB_C_Receptacle_GCT_USB4085, symbol Connector:USB_C_Receptacle_USB2.0
- removed R? (x2): 5.1k, Resistor_SMD:R_0402_1005Metric, symbol Device:R_Small
- added C?: 10uF, symbol Device:C_Small
Connections:
- net +3V3: now also C?.1; no longer IC?.8 (VDD)
- new net: C?.2, IC?.8 (VDD)
- no-connect marks 8 -> 6
Other:
- moved on the sheet: IC?

Commit message: push3schematicandpcb
Parts:
- C15: renamed from C?; footprint (none) -> Capacitor_SMD:C_0402_1005Metric
- C4: footprint (none) -> Capacitor_SMD:C_0402_1005Metric
- gave numbers to parts that had none: 1
Connections:
- no-connect marks 6 -> 36
Changed lines of the file:
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@@
   (junction (at 69.85 135.89) (diameter 0) (color 0 0 0 0)
   )
+  (no_connect (at 69.85 95.25))
+  (no_connect (at 69.85 120.65))
+  (no_connect (at 69.85 97.79))
+  (no_connect (at 135.89 107.95))
+  (no_connect (at 69.85 118.11))
+  (no_connect (at 69.85 115.57))
+  (no_connect (at 135.89 128.27))
+  (no_connect (at 69.85 80.01))
+  (no_connect (at 69.85 102.87))
+  (no_connect (at 113.03 116.84))
   (no_connect (at 185.42 104.14))
+  (no_connect (at 135.89 115.57))
+  (no_connect (at 69.85 113.03))
+  (no_connect (at 69.85 125.73))
+  (no_connect (at 69.85 72.39))
+  (no_connect (at 104.14 68.58))
+  (no_connect (at 69.85 82.55))
+  (no_connect (at 69.85 90.17))
+  (no_connect (at 69.85 123.19))
+  (no_connect (at 100.33 54.61))
+  (no_connect (at 109.22 91.44))
+  (no_connect (at 135.89 130.81))
   (no_connect (at 69.85 77.47))
+  (no_connect (at 69.85 74.93))
+  (no_connect (at 69.85 85.09))
+  (no_connect (at 69.85 100.33))
+  (no_connect (at 69.85 92.71))
   (no_connect (at 210.82 106.68))
+  (no_connect (at 135.89 118.11))
+  (no_connect (at 69.85 87.63))
+  (no_connect (at 135.89 105.41))
   (no_connect (at 135.89 113.03))
+  (no_connect (at 135.89 110.49))
+  (no_connect (at 69.85 105.41))
   (no_connect (at 135.89 123.19))
   (no_connect (at 149.86 48.26))
@@
   (symbol (lib_id "Device:C_Small") (at 214.63 100.33 0) (unit 1)
     (in_bom yes) (on_board yes) (fields_autoplaced)
-    (property "Reference" "C?" (id 0) (at 217.17 99.0662 0)
+    (property "Reference" "C15" (id 0) (at 217.17 99.0662 0)
       (effects (font (size 1.27 1.27)) (justify left))
     )
@@
       (effects (font (size 1.27 1.27)) (justify left))
     )
-    (property "Footprint" "" (id 2) (at 214.63 100.33 0)
+    (property "Footprint" "Capacitor_SMD:C_0402_1005Metric" (id 2) (at 214.63 100.33 0)
       (effects (font (size 1.27 1.27)) hide)
     )
@@
   (symbol (lib_id "power:+3.3V") (at 214.63 96.52 0) (unit 1)
     (in_bom yes) (on_board yes) (fields_autoplaced)
-    (property "Reference" "#PWR?" (id 0) (at 214.63 100.33 0)
+    (property "Reference" "#PWR0115" (id 0) (at 214.63 100.33 0)
       (effects (font (size 1.27 1.27)) hide)
     )
@@
       (effects (font (size 1.27 1.27)) (justify left))
     )
-    (property "Footprint" "" (id 2) (at 20.32 138.43 0)
+    (property "Footprint" "Capacitor_SMD:C_0402_1005Metric" (id 2) (at 20.32 138.43 0)
       (effects (font (size 1.27 1.27)) hide)
     )
@@
   (symbol (lib_id "power:GND") (at 181.61 113.03 0) (unit 1)
     (in_bom yes) (on_board yes) (fields_autoplaced)
-    (property "Reference" "#PWR?" (id 0) (at 181.61 119.38 0)
+    (property "Reference" "#PWR0114" (id 0) (at 181.61 119.38 0)
       (effects (font (size 1.27 1.27)) hide)
     )
@@
   (symbol (lib_id "chest:XTSD08GLGEAG") (at 185.42 104.14 0) (unit 1)
     (in_bom yes) (on_board yes) (fields_autoplaced)
-    (property "Reference" "IC?" (id 0) (at 198.12 96.52 0))
+    (property "Reference" "IC1" (id 0) (at 198.12 96.52 0))
     (property "Value" "XTSD08GLGEAG" (id 1) (at 198.12 99.06 0))
     (property "Footprint" "chest:SON127P800X600X95-8N" (id 2) (at 207.01 101.6 0)
@@
       (reference "#PWR0113") (unit 1) (value "GND") (footprint "")
     )
+    (path "/85da4fe0-4748-4ea0-9e9f-4695dde613ab"
+      (reference "#PWR0114") (unit 1) (value "GND") (footprint "")
+    )
+    (path "/6203f329-18ca-405c-af92-955eef11b60a"
+      (reference "#PWR0115") (unit 1) (value "+3.3V") (footprint "")
+    )
     (path "/53d816b2-077d-4de8-9c2d-91adbcde7c2a"
       (reference "#PWR0116") (unit 1) (value "+12V") (footprint "")
@@
       (reference "#PWR0151") (unit 1) (value "GND") (footprint "")
     )
-    (path "/6203f329-18ca-405c-af92-955eef11b60a"
-      (reference "#PWR?") (unit 1) (value "+3.3V") (footprint "")
-    )
-    (path "/85da4fe0-4748-4ea0-9e9f-4695dde613ab"
-      (reference "#PWR?") (unit 1) (value "GND") (footprint "")
-    )
     (path "/00000000-0000-0000-0000-00005dc1f7e5"
       (reference "3V3LED1") (unit 1) (value "3V3LED") (footprint "Resistor_SMD:R_0402_1005Metric")
@@
     )
     (path "/67acfde3-6610-495e-8efd-321e2a1a37cf"
-      (reference "C4") (unit 1) (value "10uF") (footprint "")
+      (reference "C4") (unit 1) (value "10uF") (footprint "Capacitor_SMD:C_0402_1005Metric")
     )
     (path "/e3bf37bc-a7d8-4293-a4b5-54cc127372d6"
@@
       (reference "C14") (unit 1) (value "C") (footprint "Capacitor_SMD:C_0603_1608Metric")
     )
+    (path "/0d34ff32-366e-4c28-bbbc-81ba0b7fc83b"
+      (reference "C15") (unit 1) (value "10uF") (footprint "Capacitor_SMD:C_0402_1005Metric")
+    )
     (path "/00000000-0000-0000-0000-000061925999/b893decc-b599-4714-bfdb-e8e8dc9c770c"
       (reference "C20") (unit 1) (value "10uF") (footprint "Capacitor_SMD:C_0603_1608Metric")
@@
       (reference "C37") (unit 1) (value "220 pF") (footprint "Capacitor_SMD:C_0402_1005Metric")
     )
-    (path "/0d34ff32-366e-4c28-bbbc-81ba0b7fc83b"
-      (reference "C?") (unit 1) (value "10uF") (footprint "")
-    )
     (path "/00000000-0000-0000-0000-000061925999/00000000-0000-0000-0000-000061988c8c"
       (reference "D4") (unit 1) (value "SP0503BAHT") (footprint "Package_TO_SOT_SMD:SOT-143")
@@
     )
     (path "/e70c7b52-acc8-4a8e-b292-14278aedb728"
-      (reference "IC?") (unit 1) (value "XTSD08GLGEAG") (footprint "chest:SON127P800X600X95-8N")
+      (reference "IC1") (unit 1) (value "XTSD08GLGEAG") (footprint "chest:SON127P800X600X95-8N")
     )
     (path "/00000000-0000-0000-0000-000061b03907"
