File: Ricardo-BlackBox/NewRicardoBlackBox.kicad_sch (KiCad schematic)
At the start: 37 parts, among them J1 RBUS, U1 ESP32-S3, Y1 40MHz±10ppm

Commit message: AsOf13/12/2022
Parts:
- added TP10, TP11, TP12, TP9: TestPoint, symbol Connector:TestPoint
- gave numbers to parts that had none: 2
Connections:
- net CLK: now also TP11.1
- net MISO: now also TP10.1
- net MOSI: now also TP9.1
- net NAND_CS: now also TP12.1
- net TXD: no longer R6.1
- net TXDUART: now reaches U1.50 (U0RXD/PROG/GPIO44)
- new net RXDUART: R6.1
- no-connect marks 5 -> 4
