File: Ricardo-BlackBox/can.kicad_sch (KiCad schematic)
At the start: 11 parts, among them U2 SN65HVD230

Commit message: AsOf31/01/2023
Schematic should be done, PCB beginning to be done
Changed lines of the file:
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@@
   (symbol (lib_id "Device:C") (at 171.45 88.9 90) (unit 1)
     (in_bom yes) (on_board yes) (fields_autoplaced)
-    (property "Reference" "C17" (id 0) (at 171.45 82.55 90))
-    (property "Value" "0.1uF" (id 1) (at 171.45 85.09 90))
+    (property "Reference" "C17" (id 0) (at 171.45 81.28 90))
+    (property "Value" "0.1uF" (id 1) (at 171.45 83.82 90))
     (property "Footprint" "Capacitor_SMD:C_0402_1005Metric" (id 2) (at 175.26 87.9348 0)
       (effects (font (size 1.27 1.27)) hide)
@@
   )
   (symbol_instances
+    (path "/d85aebac-c325-42de-8c8e-5349542a2954"
+      (reference "#PWR025") (unit 1) (value "GND") (footprint "")
+    )
+    (path "/49208f5a-f73e-42f1-9d7d-382d975bd991"
+      (reference "#PWR027") (unit 1) (value "GND") (footprint "")
+    )
+    (path "/54c27e2d-52b9-4197-956b-7db5f761b4df"
+      (reference "#PWR028") (unit 1) (value "GND") (footprint "")
+    )
     (path "/00000000-0000-0000-0000-000061946eb3"
       (reference "#PWR0130") (unit 1) (value "GND") (footprint "")
@@
       (reference "#PWR0131") (unit 1) (value "+3.3V") (footprint "")
     )
+    (path "/759646bf-5c31-420e-aff7-2c1a28ce32e1"
+      (reference "C15") (unit 1) (value "100nF") (footprint "Capacitor_SMD:C_0402_1005Metric")
+    )
+    (path "/06b0d844-1c7a-43fd-b8a5-ad8e34e13aac"
+      (reference "C16") (unit 1) (value "10uF") (footprint "Capacitor_SMD:C_0402_1005Metric")
+    )
+    (path "/c905e3f6-13b1-4d5f-8bb5-930cfa107996"
+      (reference "C17") (unit 1) (value "4.7nF") (footprint "Capacitor_SMD:C_0402_1005Metric")
+    )
+    (path "/23622c20-4a70-4ee7-b39c-f5519633413f"
+      (reference "C18") (unit 1) (value "220pF") (footprint "Capacitor_SMD:C_0402_1005Metric")
+    )
+    (path "/f5a97da1-282d-43a4-ae5f-607cebde55a6"
+      (reference "C19") (unit 1) (value "220pF") (footprint "Capacitor_SMD:C_0402_1005Metric")
+    )
+    (path "/4717c16e-4caf-41db-976f-f247d2a86ecc"
+      (reference "D1") (unit 1) (value "SM712_SOT23") (footprint "Package_TO_SOT_SMD:SOT-23")
+    )
+    (path "/deb2b25e-9fb0-448e-88c5-95a67db1d371"
+      (reference "JP1") (unit 1) (value "TermJP") (footprint "Jumper:SolderJumper-2_P1.3mm_Open_RoundedPad1.0x1.5mm")
+    )
+    (path "/c0a35b75-0e83-4311-add3-5a3930110d30"
+      (reference "R8") (unit 1) (value "0") (footprint "Resistor_SMD:R_0603_1608Metric")
+    )
+    (path "/c4e42d16-8dbe-42af-a61a-faa72b95fe53"
+      (reference "R9") (unit 1) (value "60") (footprint "Resistor_SMD:R_0603_1608Metric")
+    )
+    (path "/c363df37-be76-44cd-846e-5e1010ee0d3e"
+      (reference "R10") (unit 1) (value "60") (footprint "Resistor_SMD:R_0603_1608Metric")
+    )
     (path "/00000000-0000-0000-0000-000061946ec3"
