File: Ricardo-BlackBox/power.kicad_sch (KiCad schematic)
At the start: 22 parts, among them U5 LM66100, U6 LM66100, U7 MAX77827AEFD+T, U8 SC4215

Commit message: AsOf31/01/2023
Schematic should be done, PCB beginning to be done
Parts:
- removed C23: 4.7uF, Capacitor_SMD:C_0402_1005Metric, symbol Device:C_Small
- removed U5, U6: LM66100, Package_TO_SOT_SMD:SOT-23-5, symbol iclr:LTC4411
- added R14: 10k, Resistor_SMD:R_0402_1005Metric, symbol Device:R_Small
- added U3: LM66200DRLR, iclr:SOTFL50P160X60-8N, symbol iclr:LM66200DRLR
- C20: renamed from C24; value 4.7uF -> 10uF
- renumbered C25 to C21, C26 to C22, C27 to C23, C28 to C24, C29 to C25, C30 to C26, C31 to C27, R16 to R15, R17 to R16, R18 to R17, U7 to U4, U8 to U5
Connections:
- net BBIN: now also U3.2 (VOUT_1), U3.7 (VOUT_2)
- net GND: now also U3.1 (GND_1), U3.4 (~{ON}), U3.5 (GND_2)
- net RBUS_uC_V: now also U3.6 (VIN2)
- net VBUS: now also R14.1, U3.3 (VIN1)
- new net: R14.2, U3.8 (ST)
- no-connect marks 6 -> 4
Other:
- note added: "Place close together. Bridge to bypass buck-boost"
