File: Ricardo-BlackBoxNEW/Ricardo-BlackBoxNEW.kicad_sch (KiCad schematic)
At the start: 43 parts, among them IC1 XTSD08GLGEAG, J1 RBUS, U1 ESP32-S3, Y1 40MHz±10ppm

Commit message: 10_06_2023BlackBox
All files for Black Box needed are in this
Other:
- sheet USB -> UART ports: added RXD, TXD; removed none
Changed lines of the file:
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@@
     (effects (font (size 1.27 1.27)) (justify left bottom))
+  )
+  (label "TXD" (at 102.87 164.465 180) (fields_autoplaced)
+    (effects (font (size 1.27 1.27)) (justify right bottom))
   )
   (label "NAND_CS" (at 200.025 99.695 0) (fields_autoplaced)
@@
   (label "RXD" (at 29.21 43.18 0) (fields_autoplaced)
     (effects (font (size 1.27 1.27)) (justify left bottom))
+  )
+  (label "RXD" (at 102.87 162.56 180) (fields_autoplaced)
+    (effects (font (size 1.27 1.27)) (justify right bottom))
   )
   (label "CLK" (at 200.025 102.235 0) (fields_autoplaced)
@@
       (effects (font (size 1.27 1.27)) (justify right) hide)
     )
-  )
-  (hierarchical_label "RXD" (shape input) (at 99.06 164.465 180) (fields_autoplaced)
-    (effects (font (size 1.27 1.27)) (justify right))
-  )
-  (hierarchical_label "TXD" (shape input) (at 99.06 162.56 180) (fields_autoplaced)
-    (effects (font (size 1.27 1.27)) (justify right))
   )
   (symbol (lib_id "power:+3.3V") (at 30.48 182.88 0) (unit 1)
@@
       (effects (font (size 1.27 1.27)) (justify right))
     )
+    (pin "TXD" input (at 99.06 162.56 0)
+      (effects (font (size 1.27 1.27)) (justify right))
+    )
+    (pin "RXD" output (at 99.06 164.465 0)
+      (effects (font (size 1.27 1.27)) (justify right))
+    )
