File: Ricardo-BlackBoxNEW/usb-uart.kicad_sch (KiCad schematic)
At the start: 12 parts, among them IC2 CP2102N-A02-GQFN24, J2 USB_C_Receptacle_USB2.0

Commit message: 10_06_2023BlackBox
All files for Black Box needed are in this
Changed lines of the file:
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@@
-    (effects (font (size 1.27 1.27)) (justify left bottom))
-  )
-  (label "TXD" (at 211.455 80.01 0) (fields_autoplaced)
     (effects (font (size 1.27 1.27)) (justify left bottom))
   )
   (label "Data+" (at 44.45 104.14 0) (fields_autoplaced)
-    (effects (font (size 1.27 1.27)) (justify left bottom))
-  )
-  (label "RXD" (at 211.455 82.55 0) (fields_autoplaced)
     (effects (font (size 1.27 1.27)) (justify left bottom))
   )
@@
     (effects (font (size 1.27 1.27)) (justify right))
   )
+  (hierarchical_label "RXD" (shape output) (at 211.455 82.55 0) (fields_autoplaced)
+    (effects (font (size 1.27 1.27)) (justify left))
+  )
+  (hierarchical_label "TXD" (shape input) (at 211.455 80.01 0) (fields_autoplaced)
+    (effects (font (size 1.27 1.27)) (justify left))
+  )
   (hierarchical_label "Data+" (shape bidirectional) (at 44.45 104.14 180) (fields_autoplaced)
