File: Ricardo-BlackBoxNEW/Ricardo-BlackBoxNEW.kicad_pcb (KiCad board)
At the start: 4 copper layers, 53.4 x 49.6 mm, 87 parts, among them IC1 XTSD08GLGEAG, IC2 CP2102N-A02-GQFN24, J1 RBUS, J2 USB_C_Receptacle_USB2.0, U1 ESP32-S3, U2 SN65HVD230, U3 LM66200DRLR, U4 MAX77827AEFD+T, U5 SC4215, Y1 40MHz±10ppm

Commit message: RicardoBlackBox03_06_2023
Parts:
- moved R13 9.54 mm to (131.8, 115.6)
- moved USBLED1 9.45 mm to (129.5, 115.6)
- moved H4 3.53 mm to (166.4, 75.9)
- moved C10 3.49 mm to (152.5, 115.5)
- moved C11 3.49 mm to (151.5, 115.5)
- moved H3 3.02 mm to (166.2, 116.2)
- moved TP8 2.91 mm to (162.3, 73.7)
- moved R3 2.28 mm to (147.6, 118.1)
- moved C8 2.21 mm to (147.6, 117.0)
- moved R4 1.98 mm to (156.1, 95.7)
- moved C13 1.98 mm to (153.6, 95.1)
- moved C3 1.98 mm to (147.3, 107.9)
- moved C9 1.98 mm to (147.2, 98.2)
- moved R7 1.98 mm to (160.7, 91.5)
- moved TP12 1.98 mm to (166.6, 106.7)
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Routing:
- net VBUS: track 55.9 -> 103.3 mm, vias 4 -> 2
- net /Data+: track 37.3 -> 80.1 mm
- net /Data-: track 41.3 -> 71.3 mm
- net GND: track 81.1 -> 66.1 mm, vias 30 -> 18
- net /Power/LX1: track 0.00 -> 14.1 mm
- net /Power/LX2: track 0.00 -> 11.6 mm
- net /Power/BBIN: track 3.68 -> 14.1 mm
- net +3V3: track 82.3 -> 85.7 mm
- net +12V: track 40.5 -> 38.6 mm
- net /TXD: track 22.6 -> 20.7 mm
- net /RXD: track 28.6 -> 26.8 mm
- net RBUS_uC_V: track 18.5 -> 16.8 mm
- net Net-(J2-PadA5): track 4.06 -> 5.07 mm
- net Net-(J2-PadB5): track 1.87 -> 2.88 mm
- net /Power/BBOUT: track 16.7 -> 16.1 mm
- added copper zone on In1.Cu, net +3V3
- added copper zone on In2.Cu, net GND
Other:
- board size 53.4 x 49.6 mm -> 50.9 x 47.8 mm

Commit message: 03/06/2023RicardoBlackBoxAfterICLRMeeting
13:31
Parts:
- moved H1 0.61 mm to (123.8, 115.8)
- moved H4 0.54 mm to (165.9, 75.7)
- moved H2 0.49 mm to (123.4, 75.9)
- moved TP6 0.47 mm to (143.2, 82.5)
- moved J2 0.46 mm to (124.0, 101.3)
- moved TP8 0.42 mm to (161.9, 73.8)
- moved TP1 0.32 mm to (129.2, 110.0)
- moved H3 0.31 mm to (165.9, 116.2)
- moved TP12 0.18 mm to (166.8, 106.7)
- moved C2 0.14 mm to (147.1, 105.3)
Routing:
- net /Power/LX1: track 14.1 -> 0.04 mm
- net /Power/LX2: track 11.6 -> 0.44 mm
- net GND: track 66.1 -> 73.2 mm, vias 18 -> 16
- net /Power/BBIN: track 14.1 -> 10.5 mm
- net /CHIP_PU: track 12.5 -> 9.20 mm
- net VBUS: track 103.3 -> 102.1 mm
- net +3V3: track 85.7 -> 84.7 mm
- net /Data+: track 80.1 -> 79.1 mm
Other:
- board size 50.9 x 47.8 mm -> 49.8 x 47.8 mm

Commit message: 10_06_2023BlackBox
All files for Black Box needed are in this
Parts:
- moved R7 6.76 mm to (153.9, 91.6)
- moved 12VLED1 6.69 mm to (151.9, 91.6)
- moved ENJUMPER1 4.96 mm to (141.6, 109.8)
- moved BOOTJUMPER1 4.91 mm to (141.6, 113.6)
- moved TP4 3.45 mm to (146.6, 77.5)
- moved C8 2.48 mm to (146.9, 114.6)
- moved R3 2.42 mm to (147.0, 115.8)
- moved H3 1.70 mm to (165.3, 114.7)
- moved H1 1.52 mm to (123.9, 114.2)
- moved TP10 1.20 mm to (159.2, 99.6)
- moved L2 1.09 mm to (151.7, 101.4)
- moved U2 0.69 mm to (130.9, 91.3)
- moved R8 0.67 mm to (134.2, 87.8)
- moved C13 0.42 mm to (153.9, 95.3)
- moved C16 0.37 mm to (126.4, 92.4)
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Connections:
- IC2 pad 20: /RXD -> /TXD
- IC2 pad 21: /TXD -> /RXD
Routing:
- net +12V: track 38.6 -> 32.2 mm
- net /CHIP_PU: track 9.20 -> 13.0 mm
- net GND: track 73.2 -> 76.6 mm, vias 16 -> 18
- net /BOOT: track 18.7 -> 21.9 mm
- net Net-(C14-Pad1): track 8.25 -> 6.72 mm
- net /CAN-BUS/Vref: track 7.64 -> 6.25 mm
- net Net-(U1-XTAL_P): track 1.95 -> 3.12 mm
- net /Power/BBIN: track 10.5 -> 9.39 mm
- net +3V3: track 84.7 -> 85.8 mm
- net /CAN-: track 34.5 -> 35.3 mm
- net /Data+: track 79.1 -> 78.4 mm
- net /CAN+: track 26.5 -> 27.1 mm
- net /RXD: track 26.8 -> 27.3 mm, vias 4 -> 3
Other:
- board size 49.8 x 47.8 mm -> 49.8 x 46.6 mm

Commit message: Black_Box_20/06/2023_THIS_HAS_ALL_FOLDER_HAS_FILES
This folder has the board up to date
Parts:
- moved R13 2.38 mm to (130.4, 113.7)
- moved USBLED1 2.23 mm to (128.4, 113.7)
- moved C15 0.97 mm to (124.3, 92.3)
- moved C16 0.67 mm to (125.8, 92.3)
- moved TP2 0.50 mm to (131.5, 109.5)
- moved TP1 0.20 mm to (129.2, 109.8)
Routing:
- net VBUS: track 102.0 -> 97.7 mm
- net +3V3: track 85.8 -> 87.0 mm
- net /Data+: track 78.4 -> 77.9 mm

Commit message: BlackBox_20_06_2023_ThisFolderHasAllTheFilesNeeded
Parts:
- moved TP13 0.77 mm to (159.6, 111.8)
- moved TP3 0.59 mm to (162.4, 103.4)
- moved IC1 0.50 mm to (163.1, 106.3)
Routing:
- net +3V3: track 87.0 -> 85.9 mm
- net /NAND_CS: track 15.0 -> 15.7 mm
- net /MISO: track 9.29 -> 8.96 mm, vias 3 -> 2
