File: Ricardo-BlackBoxNEWFinal/can.kicad_sch (KiCad schematic)
At the start: 11 parts, among them U2 SN65HVD230

Commit message: RicardoBlackBoxFinal_20_08_2023
Parts:
- removed C18, C19: 220pF, Capacitor_SMD:C_0402_1005Metric, symbol Device:C_Small
- C17: value 0.1uF -> 47nF
- R10, R9: footprint Resistor_SMD:R_0402_1005Metric -> Resistor_SMD:R_0603_1608Metric
Changed lines of the file:
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@@
-    (stroke (width 0) (type default))
-  )
-  (wire (pts (xy 175.26 85.09) (xy 175.26 88.9))
     (stroke (width 0) (type default))
   )
@@
     )
   )
-  (symbol (lib_id "Device:C_Small") (at 175.26 82.55 180) (unit 1)
-    (in_bom yes) (on_board yes) (dnp no)
-    (property "Reference" "C18" (at 173.99 74.93 0)
-      (effects (font (size 1.27 1.27)) (justify right))
-    )
-    (property "Value" "220pF" (at 173.99 77.47 0)
-      (effects (font (size 1.27 1.27)) (justify right))
-    )
-    (property "Footprint" "Capacitor_SMD:C_0402_1005Metric" (at 175.26 82.55 0)
-      (effects (font (size 1.27 1.27)) hide)
-    )
-    (property "Datasheet" "~" (at 175.26 82.55 0)
-      (effects (font (size 1.27 1.27)) hide)
-    )
-    (pin "1")
-    (pin "2")
-    (instances
-      (project "Ricardo-BlackBoxNEWFinal"
-        (path "/7db990e4-92e1-4f99-b4d2-435bbec1ba83/00000000-0000-0000-0000-000061942b9a"
-          (reference "C18") (unit 1)
-        )
-      )
-    )
-  )
   (symbol (lib_id "Diode:SM712_SOT23") (at 186.69 88.9 270) (unit 1)
     (in_bom yes) (on_board yes) (dnp no) (fields_autoplaced)
@@
         (path "/7db990e4-92e1-4f99-b4d2-435bbec1ba83/00000000-0000-0000-0000-000061942b9a"
           (reference "#PWR027") (unit 1)
-        )
-      )
-    )
-  )
-  (symbol (lib_id "power:GND") (at 175.26 102.87 0) (unit 1)
-    (in_bom yes) (on_board yes) (dnp no) (fields_autoplaced)
-    (property "Reference" "#PWR028" (at 175.26 109.22 0)
-      (effects (font (size 1.27 1.27)) hide)
-    )
-    (property "Value" "GND" (at 175.26 106.68 0)
-      (effects (font (size 1.27 1.27)))
-    )
-    (property "Footprint" "" (at 175.26 102.87 0)
-      (effects (font (size 1.27 1.27)) hide)
-    )
-    (property "Datasheet" "" (at 175.26 102.87 0)
-      (effects (font (size 1.27 1.27)) hide)
-    )
-    (pin "1")
-    (instances
-      (project "Ricardo-BlackBoxNEWFinal"
-        (path "/7db990e4-92e1-4f99-b4d2-435bbec1ba83/00000000-0000-0000-0000-000061942b9a"
-          (reference "#PWR028") (unit 1)
         )
       )
@@
       (effects (font (size 1.27 1.27)) (justify left))
     )
-    (property "Footprint" "Resistor_SMD:R_0402_1005Metric" (at 165.862 93.98 90)
+    (property "Footprint" "Resistor_SMD:R_0603_1608Metric" (at 165.862 93.98 90)
       (effects (font (size 1.27 1.27)) hide)
     )
@@
       (effects (font (size 1.27 1.27)) (justify left))
     )
-    (property "Footprint" "Resistor_SMD:R_0402_1005Metric" (at 165.862 83.82 90)
+    (property "Footprint" "Resistor_SMD:R_0603_1608Metric" (at 165.862 83.82 90)
       (effects (font (size 1.27 1.27)) hide)
     )
@@
   (symbol (lib_id "Device:C") (at 171.45 88.9 90) (unit 1)
     (in_bom yes) (on_board yes) (dnp no) (fields_autoplaced)
-    (property "Reference" "C17" (at 171.45 81.28 90)
-      (effects (font (size 1.27 1.27)))
-    )
-    (property "Value" "0.1uF" (at 171.45 83.82 90)
+    (property "Reference" "C17" (at 171.45 82.55 90)
+      (effects (font (size 1.27 1.27)))
+    )
+    (property "Value" "47nF" (at 171.45 85.09 90)
       (effects (font (size 1.27 1.27)))
     )
@@
         )
       )
-    )
-  )
-  (symbol (lib_id "Device:C_Small") (at 175.26 100.33 180) (unit 1)
-    (in_bom yes) (on_board yes) (dnp no) (fields_autoplaced)
-    (property "Reference" "C19" (at 177.8 99.0535 0)
-      (effects (font (size 1.27 1.27)) (justify right))
-    )
-    (property "Value" "220pF" (at 177.8 101.5935 0)
-      (effects (font (size 1.27 1.27)) (justify right))
-    )
-    (property "Footprint" "Capacitor_SMD:C_0402_1005Metric" (at 175.26 100.33 0)
-      (effects (font (size 1.27 1.27)) hide)
-    )
-    (property "Datasheet" "~" (at 175.26 100.33 0)
-      (effects (font (size 1.27 1.27)) hide)
-    )
-    (pin "1")
-    (pin "2")
-    (instances
-      (project "Ricardo-BlackBoxNEWFinal"
-        (path "/7db990e4-92e1-4f99-b4d2-435bbec1ba83/00000000-0000-0000-0000-000061942b9a"
-          (reference "C19") (unit 1)
-        )
-      )
