File: Ricardo-BlackBoxNEWFinal/usb-uart.kicad_sch (KiCad schematic)
At the start: 12 parts, among them IC2 CP2102N-A02-GQFN24, J2 USB_C_Receptacle_USB2.0

Commit message: Ricardo-BlackBoxNEWFinal_14_08_2023
Connections:
- net Data+: no longer J2.B6 (D+)
- net Data-: no longer J2.B7 (D-)
- no-connect marks 18 -> 20
Changed lines of the file:
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@@
 (kicad_sch (version 20230121) (generator eeschema)
   (paper "A4")
-  (junction (at 127 116.84) (diameter 0) (color 0 0 0 0)
-  )
   (junction (at 143.51 97.79) (diameter 0) (color 0 0 0 0)
   )
@@
   (junction (at 146.05 111.76) (diameter 0) (color 0 0 0 0)
   )
-  (junction (at 127 111.76) (diameter 0) (color 0 0 0 0)
-  )
   (junction (at 107.95 135.89) (diameter 0) (color 0 0 0 0)
   )
@@
   (junction (at 148.59 116.84) (diameter 0) (color 0 0 0 0)
   )
+  (no_connect (at 127 113.03))
   (no_connect (at 211.455 92.71))
   (no_connect (at 165.735 100.33))
@@
   (no_connect (at 127 125.73))
   (no_connect (at 211.455 113.03))
+  (no_connect (at 127 118.11))
   (no_connect (at 211.455 97.79))
   (no_connect (at 211.455 87.63))
@@
   )
   (wire (pts (xy 44.45 104.14) (xy 52.07 104.14))
-    (stroke (width 0) (type default))
-  )
-  (wire (pts (xy 127 116.84) (xy 127 118.11))
     (stroke (width 0) (type default))
   )
@@
     (stroke (width 0) (type default))
   )
+  (wire (pts (xy 148.59 115.57) (xy 148.59 116.84))
+    (stroke (width 0) (type default))
+  )
   (wire (pts (xy 127 102.87) (xy 132.08 102.87))
     (stroke (width 0) (type default))
@@
     (stroke (width 0) (type default))
   )
-  (wire (pts (xy 127 115.57) (xy 127 116.84))
-    (stroke (width 0) (type default))
-  )
   (wire (pts (xy 149.225 72.39) (xy 165.735 72.39))
-    (stroke (width 0) (type default))
-  )
-  (wire (pts (xy 127 113.03) (xy 127 111.76))
     (stroke (width 0) (type default))
   )
@@
     (stroke (width 0) (type default))
   )
-  (wire (pts (xy 127 116.84) (xy 148.59 116.84))
+  (wire (pts (xy 127 115.57) (xy 148.59 115.57))
     (stroke (width 0) (type default))
   )

Commit message: Ricardo-BlackBoxFinal_15_08_2023
Parts:
- removed IC2: CP2102N-A02-GQFN24, iclr:QFN50P400X400X80-25N, symbol iclr:CP2102N-A02-GQFN24
- removed R18: 22.1k, Resistor_SMD:R_0402_1005Metric, symbol Device:R_Small
- removed R19: 47.5k, Resistor_SMD:R_0402_1005Metric, symbol Device:R_Small
Connections:
- net Data+: now also D2.3 (K), J2.B6 (D+); no longer D2.4 (K)
- net Data-: now also D2.4 (K), J2.B7 (D-); no longer D2.3 (K)
- no-connect marks 20 -> 2

Commit message: RicardoBlackBoxFinal_20_08_2023
Parts:
- removed TP14: TestPoint, TestPoint:TestPoint_Pad_D1.0mm, symbol Connector:TestPoint
Changed lines of the file:
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@@
-    (stroke (width 0) (type default))
-  )
-  (wire (pts (xy 48.26 108.585) (xy 52.07 108.585))
     (stroke (width 0) (type default))
   )
@@
   (label "Data-" (at 44.45 99.06 0) (fields_autoplaced)
     (effects (font (size 1.27 1.27)) (justify left bottom))
-  )
-  (label "VBUS" (at 48.26 108.585 180) (fields_autoplaced)
-    (effects (font (size 1.27 1.27)) (justify right bottom))
   )
   (label "Data+" (at 146.05 127 90) (fields_autoplaced)
@@
         )
       )
-    )
-  )
-  (symbol (lib_id "Connector:TestPoint") (at 52.07 108.585 270) (unit 1)
-    (in_bom yes) (on_board yes) (dnp no) (fields_autoplaced)
-    (property "Reference" "TP14" (at 57.15 107.3149 90)
-      (effects (font (size 1.27 1.27)) (justify left))
-    )
-    (property "Value" "TestPoint" (at 57.15 109.8549 90)
-      (effects (font (size 1.27 1.27)) (justify left))
-    )
-    (property "Footprint" "TestPoint:TestPoint_Pad_D1.0mm" (at 52.07 113.665 0)
-      (effects (font (size 1.27 1.27)) hide)
-    )
-    (property "Datasheet" "~" (at 52.07 113.665 0)
-      (effects (font (size 1.27 1.27)) hide)
-    )
-    (pin "1")
-    (instances
-      (project "Ricardo-BlackBoxNEWFinal"
-        (path "/7db990e4-92e1-4f99-b4d2-435bbec1ba83/00000000-0000-0000-0000-000061925999"
-          (reference "TP14") (unit 1)
-        )
-      )
