File: Ricardo-BlackBoxNEWFinal/Ricardo-BlackBoxNEWFinal.kicad_pcb (KiCad board)
At the start: 4 copper layers, 44 x 50 mm, 87 parts, among them IC1 XTSD08GLGEAG, IC2 CP2102N-A02-GQFN24, J1 RBUS, J2 USB_C_Receptacle_USB2.0, U1 ESP32-S3, U2 SN65HVD230, U3 LM66200DRLR, U4 MAX77827AEFD+T, U5 SC4215, Y1 40MHz±10ppm

Commit message: RicardoBlackBoxNEWFinal_13_08_2023
Parts:
- moved TP6 35.2 mm to (156.2, 88.6)
- moved C11 16.7 mm to (152.2, 107.5), turned to 0 degrees
- moved Y1 9.11 mm to (151.5, 101.6)
- moved C28 7.41 mm to (152.6, 113.9)
- moved C13 6.24 mm to (151.6, 98.5)
- moved C14 5.33 mm to (151.8, 103.6)
- moved C10 4.32 mm to (144.4, 116.2)
- moved TP12 4.01 mm to (156.7, 112.5)
- moved TP1 3.86 mm to (130.2, 106.0)
- moved TP11 3.52 mm to (155.6, 109.6)
- moved L2 3.33 mm to (149.9, 104.2)
- moved TP13 2.58 mm to (152.4, 116.5)
- moved IC1 2.50 mm to (153.5, 112.0)
- moved C8 2.44 mm to (136.5, 116.5)
- moved TP3 2.21 mm to (153.4, 109.5)
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Connections:
- U1 pad 13: unconnected-(U1-GPIO8/ADC1_CH7-Pad13) -> /CAN_RX
- U1 pad 14: unconnected-(U1-GPIO9/ADC1_CH8-Pad14) -> /CAN_TX
Routing:
- net /CAN_TX: track 0.00 -> 39.9 mm, vias 0 -> 2
- net /CAN_RX: track 0.00 -> 30.7 mm, vias 0 -> 2
- net GND: track 78.9 -> 65.5 mm
- net Net-(U1-XTAL_N): track 26.2 -> 18.5 mm
- net Net-(C14-Pad1): track 10.7 -> 3.12 mm
- net +3V3: track 97.9 -> 92.1 mm, vias 10 -> 11
- net /CAN-: track 31.9 -> 37.1 mm
- net Net-(IC1-VDD): track 6.30 -> 1.37 mm, vias 2 -> 0
- net /NAND_CS: track 18.3 -> 13.5 mm, vias 2 -> 0
- net /CAN+: track 26.2 -> 30.3 mm
- net VBUS: track 94.4 -> 98.0 mm, vias 2 -> 4
- net Net-(U1-XTAL_P): track 10.3 -> 6.84 mm
- net /CAN-BUS/Vref: track 7.27 -> 10.5 mm
- net /Data+: track 71.7 -> 68.7 mm, vias 5 -> 4
- net /CLK: track 16.1 -> 18.8 mm
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Other:
- outline, holes or cut-outs redrawn

Commit message: Ricardo-BlackBoxNEWFinal_14_08_2023
Parts:
- C13, C14: value C -> 11pF
- moved D1 6.54 mm to (136.5, 86.0), turned to -90 degrees
- moved TP1 5.71 mm to (135.7, 104.7), turned to 90 degrees
- moved C19 5.34 mm to (137.7, 88.5), turned to 180 degrees
- moved C18 3.73 mm to (135.0, 88.5), turned to 0 degrees
- moved R10 3.43 mm to (138.1, 89.7), turned to 0 degrees
- moved TP10 3.22 mm to (159.6, 97.1)
- moved R8 3.04 mm to (121.0, 87.3), turned to 90 degrees
- moved R9 2.72 mm to (134.2, 89.9)
- moved TP9 2.57 mm to (160.6, 101.1)
- moved R6 2.28 mm to (158.6, 103.4)
- moved TXLED1 2.19 mm to (158.6, 101.1)
- moved C13 1.93 mm to (153.0, 99.9), turned to 180 degrees
- moved R19 1.93 mm to (131.7, 99.2), turned to 180 degrees
- moved R11 1.88 mm to (129.6, 99.7)
- moved JP1 1.71 mm to (135.9, 91.1), turned to 90 degrees
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Connections:
- J2 pad B6: /Data+ -> unconnected-(J2-D+-PadB6)
- J2 pad B7: /Data- -> unconnected-(J2-D--PadB7)
Routing:
- net /CAN_RX: track 30.7 -> 42.0 mm, vias 2 -> 0
- net /TXD: track 21.1 -> 30.1 mm
- net /Data-: track 64.7 -> 58.0 mm
- net /RXD: track 37.5 -> 44.1 mm
- net /Data+: track 68.7 -> 62.6 mm, vias 4 -> 2
- net /CAN-: track 37.1 -> 32.4 mm
- net /CAN-BUS/Vref: track 10.5 -> 14.4 mm
- net /CAN_TX: track 39.9 -> 43.7 mm, vias 2 -> 0
- net GND: track 65.5 -> 62.0 mm, vias 20 -> 37
- net /CAN+: track 30.3 -> 32.5 mm
- net VBUS: track 98.0 -> 99.9 mm, vias 4 -> 6
- net Net-(J2-CC1): track 4.63 -> 2.71 mm
- net Net-(U1-U0TXD/PROG/GPIO43): track 12.0 -> 13.6 mm
- net Net-(TXLED1-A): track 1.81 -> 3.28 mm
- net Net-(U1-XTAL_P): track 6.84 -> 5.74 mm
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
Commit message: Ricardo-BlackBoxFinal_15_08_2023
Parts:
- removed IC2: CP2102N-A02-GQFN24, iclr:QFN50P400X400X80-25N
- removed R18: 22.1k, Resistor_SMD:R_0402_1005Metric
- removed R19: 47.5k, Resistor_SMD:R_0402_1005Metric
- added G***: LOGO, LOGO, F.Cu at (128.7, 45.1)
- IC1: footprint iclr:SOTFL50P160X60-8N -> iclr:SON127P800X600X95-8N
- moved H3 83.3 mm to (118.5, 45.2)
- moved R3 69.5 mm to (142.0, 48.3), turned to -90 degrees
- moved C8 68.9 mm to (140.8, 47.7), turned to 90 degrees
- moved BOOTJUMPER1 68.6 mm to (138.4, 49.2)
- moved TP13 65.7 mm to (169.6, 53.0)
- moved ENJUMPER1 65.7 mm to (145.6, 46.1), turned to 180 degrees
- moved USBLED1 62.0 mm to (169.1, 65.7), turned to 180 degrees
- moved TP12 61.4 mm to (172.0, 53.0)
- moved R13 60.1 mm to (167.0, 65.7), turned to 0 degrees
- moved C3 58.8 mm to (148.1, 47.0), turned to 90 degrees
- moved TP11 57.9 mm to (167.4, 53.0)
- moved TP3 57.6 mm to (165.3, 53.1)
- moved TP2 56.5 mm to (163.0, 63.6)
- moved IC1 56.5 mm to (168.0, 57.4)
- moved R1 54.8 mm to (145.2, 49.6)
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Connections:
- D2 pad 3: /Data- -> /Data+
- D2 pad 4: /Data+ -> /Data-
- J2 pad B6: unconnected-(J2-D+-PadB6) -> /Data+
- J2 pad B7: unconnected-(J2-D--PadB7) -> /Data-
Routing:
- net VBUS: track 99.9 -> 46.6 mm, vias 6 -> 2
- net /Data+: track 62.6 -> 10.6 mm, vias 2 -> 0
- net +3V3: track 91.5 -> 42.7 mm, vias 11 -> 10
- net /Data-: track 58.0 -> 11.8 mm
- net +12V: track 31.8 -> 72.4 mm
- net /RXD: track 44.1 -> 8.09 mm, vias 3 -> 0
- net GND: track 62.0 -> 28.5 mm, vias 37 -> 52
- net /CAN_TX: track 43.7 -> 11.4 mm
- net /CAN_RX: track 42.0 -> 10.3 mm
- net /TXD: track 30.1 -> 5.06 mm, vias 2 -> 0
- net Net-(U1-XTAL_N): track 18.1 -> 6.24 mm
- net Net-(U1-U0TXD/PROG/GPIO43): track 13.6 -> 4.69 mm
- net Net-(U1-LNA_IN/RF): track 9.57 -> 1.26 mm
- net RBUS_uC_V: track 31.0 -> 37.6 mm
- net /CAN+: track 32.5 -> 27.7 mm
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- added copper zone on B.Cu, net GND
- removed copper zone on In2.Cu, net GND
Other:
- board size 44 x 50 mm -> 62 x 33 mm

Commit message: RicardoBlackBoxFinal(2)_15_08_2023
Parts:
- moved G*** 2.58 mm to (126.1, 45.0)
- moved R12 0.11 mm to (163.2, 65.6)
Routing:
- net /CAN+: track 27.7 -> 28.3 mm

Commit message: RicardoBlackBoxFinal_15_08_2023_(3)
Parts:
- moved TP6 4.76 mm to (147.7, 62.8), turned to 180 degrees
- moved C9 4.37 mm to (154.2, 53.7), turned to 180 degrees
- moved R5 1.54 mm to (152.9, 55.3), turned to 90 degrees
- moved C7 0.87 mm to (153.5, 52.7)
Routing:
- net +3V3: track 42.7 -> 40.9 mm
- net /BOOT: track 25.3 -> 26.8 mm
- net Net-(C6-Pad1): track 9.87 -> 11.2 mm
- net /CHIP_PU: track 22.5 -> 23.7 mm
- net GND: vias 52 -> 51
Other:
- board text added: "S.I.R.I.U.S. by Benedek Horvath Trinidad"

Commit message: RicardoBlackBox_15_08_2023_(4)
Parts:
- moved C10 3.21 mm to (157.7, 63.1)
- moved TP1 1.41 mm to (155.5, 64.8)
- moved TP5 0.57 mm to (144.9, 62.1)
Routing:
- net +3V3: track 40.9 -> 37.6 mm
- net GND: track 28.5 -> 26.9 mm, vias 51 -> 45
- net /Data-: track 11.8 -> 13.2 mm
- net +12V: track 72.4 -> 71.5 mm

Commit message: RicardoBlackBoxFinal_20_08_2023
Parts:
- removed 12VLED1: 12V_LED, Resistor_SMD:R_0402_1005Metric
- removed C18, C19: 220pF, Capacitor_SMD:C_0402_1005Metric
- removed TP14: TestPoint, TestPoint:TestPoint_Pad_D1.0mm
- added C29: 0.1uF, Capacitor_SMD:C_0402_1005Metric, F.Cu at (173.3, 55.2)
- added G***: LOGO, LOGO, B.Cu at (148.7, 59.8)
- C17: value 0.1uF -> 47nF
- R10, R9: footprint Resistor_SMD:R_0402_1005Metric -> Resistor_SMD:R_0603_1608Metric
- U1: footprint Package_DFN_QFN:QFN-56-1EP_7x7mm_P0.4mm_EP5.6x5.6mm -> iclr:QFN40P700X700X90-57N
- moved TP12 11.0 mm to (165.6, 62.0)
- moved TP11 9.37 mm to (170.5, 61.9)
- moved C5 9.27 mm to (150.6, 57.6)
- moved BOOTJUMPER1 9.23 mm to (147.3, 46.7), turned to 180 degrees
- moved C28 9.20 mm to (173.3, 57.8), turned to -90 degrees
- moved C4 8.91 mm to (150.6, 56.2)
- moved TP13 8.89 mm to (168.0, 61.8)
- moved C1 8.62 mm to (150.6, 54.8)
- moved L1 8.52 mm to (152.6, 57.7)
- moved C2 7.29 mm to (152.2, 50.4), turned to 0 degrees
- moved C8 7.12 mm to (147.4, 50.5), turned to 180 degrees
- moved R1 7.02 mm to (152.2, 49.4), turned to 180 degrees
- moved C6 6.45 mm to (152.6, 56.7)
- moved C3 6.09 mm to (152.2, 51.5), turned to 0 degrees
- moved ENJUMPER1 5.54 mm to (151.1, 46.7)
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Connections:
- C28 pad 1: +3V3 -> Net-(IC1-VDD)
- C28 pad 2: Net-(IC1-VDD) -> GND
- R7 pad 2: Net-(12VLED1-A) -> GND
Routing:
- net VBUS: track 46.6 -> 70.6 mm
- net /MOSI: track 5.22 -> 26.1 mm
- net /CLK: track 19.4 -> 7.79 mm
- net /MISO: track 7.31 -> 15.3 mm
- net +12V: track 71.5 -> 79.2 mm
- net Net-(C6-Pad1): track 11.2 -> 3.68 mm
- net +3V3: track 37.6 -> 31.7 mm, vias 10 -> 12
- net /NAND_CS: track 14.5 -> 10.1 mm
- net GND: track 26.9 -> 31.1 mm, vias 45 -> 47
- net /CAN_TX: track 11.4 -> 14.4 mm
- net /BOOT: track 26.8 -> 23.9 mm
- net /CAN-: track 28.5 -> 30.5 mm
- net /CAN_RX: track 10.3 -> 12.1 mm
- net Net-(JP1-B): track 3.91 -> 5.50 mm
- net Net-(IC1-VDD): track 1.88 -> 3.27 mm
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
Commit message: RicardoBlackBox_20_08_2023(2)
Parts:
- removed R7: 3k, Resistor_SMD:R_0402_1005Metric
- moved C28 2.18 mm to (174.6, 56.0)
- moved C29 0.86 mm to (173.5, 56.0)
- moved TP2 0.40 mm to (163.0, 62.4)
- moved TP12 0.24 mm to (165.5, 61.8)
- moved C17 0.24 mm to (133.4, 55.4)
- moved R9 0.21 mm to (134.7, 57.5)
- moved C1 0.07 mm to (150.5, 54.8)
- moved R10 0.06 mm to (134.7, 53.4)
Connections:
- C28 pad 1: Net-(IC1-VDD) -> +3V3
- C29 pad 2: Net-(IC1-VDD) -> GND
- IC1 pad 8: Net-(IC1-VDD) -> +3V3
Routing:
- net +12V: track 79.2 -> 0.00 mm, vias 2 -> 0
- net +3V3: track 31.7 -> 35.7 mm, vias 12 -> 11
- net Net-(IC1-VDD): track 3.27 -> 0.00 mm
