File: Ricardo-BlackBoxNEWFinal/Ricardo-BlackBoxNEWFinal.kicad_sch (KiCad schematic)
At the start: 43 parts, among them IC1 XTSD08GLGEAG, J1 RBUS, U1 ESP32-S3, Y1 40MHz±10ppm

Commit message: RicardoBlackBoxNEWFinal_13_08_2023
Connections:
- net CAN_RX: now also U1.13 (GPIO8/ADC1_CH7)
- net CAN_TX: now also U1.14 (GPIO9/ADC1_CH8)
- no-connect marks 39 -> 37

Commit message: Ricardo-BlackBoxNEWFinal_14_08_2023
Parts:
- C13, C14: value C -> 11pF
Changed lines of the file:
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@@
       (effects (font (size 1.27 1.27)) (justify left))
     )
-    (property "Value" "C" (at 165.1 144.5514 90)
+    (property "Value" "11pF" (at 165.1 144.5514 90)
       (effects (font (size 1.27 1.27)) (justify left))
     )
@@
       (effects (font (size 1.27 1.27)) (justify left))
     )
-    (property "Value" "C" (at 163.83 124.2314 90)
+    (property "Value" "11pF" (at 163.83 124.2314 90)
       (effects (font (size 1.27 1.27)) (justify left))
     )

Commit message: Ricardo-BlackBoxFinal_15_08_2023
Parts:
- IC1: footprint iclr:SOTFL50P160X60-8N -> iclr:SON127P800X600X95-8N
Changed lines of the file:
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@@
       (effects (font (size 1.27 1.27)))
     )
-    (property "Footprint" "iclr:SOTFL50P160X60-8N" (at 226.695 94.615 0)
+    (property "Footprint" "iclr:SON127P800X600X95-8N" (at 226.695 94.615 0)
       (effects (font (size 1.27 1.27)) (justify left) hide)
     )

Commit message: RicardoBlackBoxFinal_20_08_2023
Parts:
- removed 12VLED1: 12V_LED, Resistor_SMD:R_0402_1005Metric, symbol Device:LED_Small
- added C29: 0.1uF, Capacitor_SMD:C_0402_1005Metric, symbol Device:C_Small
- U1: footprint Package_DFN_QFN:QFN-56-1EP_7x7mm_P0.4mm_EP5.6x5.6mm -> iclr:QFN40P700X700X90-57N
Connections:
- net +3V3: now also C29.1; no longer C28.1
- net GND: now also C28.2, R7.2
- net at IC1.8 (VDD): now also C28.1, C29.2; no longer C28.2
Other:
- moved on the sheet: C28
Changed lines of the file:
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@@
   (junction (at 58.42 26.67) (diameter 0) (color 0 0 0 0)
+  )
+  (junction (at 240.665 97.155) (diameter 0) (color 0 0 0 0)
   )
   (junction (at 30.48 191.77) (diameter 0) (color 0 0 0 0)
@@
   (no_connect (at 135.89 82.55))
   (no_connect (at 135.89 105.41))
-  (wire (pts (xy 234.315 95.885) (xy 234.315 97.155))
-    (stroke (width 0) (type default))
-  )
   (wire (pts (xy 200.025 102.235) (xy 205.105 102.235))
     (stroke (width 0) (type default))
@@
     (stroke (width 0) (type default))
   )
-  (wire (pts (xy 60.96 26.67) (xy 58.42 26.67))
+  (wire (pts (xy 58.42 26.67) (xy 66.04 26.67))
     (stroke (width 0) (type default))
   )
@@
     (stroke (width 0) (type default))
   )
+  (wire (pts (xy 240.665 99.695) (xy 240.665 97.155))
+    (stroke (width 0) (type default))
+  )
   (wire (pts (xy 58.42 21.59) (xy 57.15 21.59))
     (stroke (width 0) (type default))
@@
     (stroke (width 0) (type default))
   )
-  (wire (pts (xy 234.315 97.155) (xy 230.505 97.155))
-    (stroke (width 0) (type default))
-  )
   (wire (pts (xy 16.51 170.18) (xy 16.51 171.45))
     (stroke (width 0) (type default))
@@
     (stroke (width 0) (type default))
   )
+  (wire (pts (xy 230.505 97.155) (xy 240.665 97.155))
+    (stroke (width 0) (type default))
+  )
   (wire (pts (xy 59.69 62.23) (xy 63.5 62.23))
     (stroke (width 0) (type default))
@@
     (stroke (width 0) (type default))
   )
+  (wire (pts (xy 240.665 97.155) (xy 240.665 95.885))
+    (stroke (width 0) (type default))
+  )
+  (wire (pts (xy 240.665 90.805) (xy 240.665 88.9))
+    (stroke (width 0) (type default))
+  )
   (wire (pts (xy 59.69 67.31) (xy 69.85 67.31))
     (stroke (width 0) (type default))
@@
   )
   (wire (pts (xy 58.42 26.67) (xy 58.42 40.64))
-    (stroke (width 0) (type default))
-  )
-  (wire (pts (xy 234.315 89.535) (xy 234.315 90.805))
     (stroke (width 0) (type default))
   )
@@
     )
   )
-  (symbol (lib_id "Device:LED_Small") (at 63.5 26.67 0) (unit 1)
-    (in_bom yes) (on_board yes) (dnp no)
-    (property "Reference" "12VLED1" (at 63.5 31.877 0)
-      (effects (font (size 1.27 1.27)))
-    )
-    (property "Value" "12V_LED" (at 63.5 29.5656 0)
-      (effects (font (size 1.27 1.27)))
-    )
-    (property "Footprint" "Resistor_SMD:R_0402_1005Metric" (at 63.5 26.67 90)
-      (effects (font (size 1.27 1.27)) hide)
-    )
-    (property "Datasheet" "~" (at 63.5 26.67 90)
-      (effects (font (size 1.27 1.27)) hide)
-    )
-    (pin "1")
-    (pin "2")
-    (instances
-      (project "Ricardo-BlackBoxNEWFinal"
-        (path "/7db990e4-92e1-4f99-b4d2-435bbec1ba83"
-          (reference "12VLED1") (unit 1)
-        )
-      )
-    )
-  )
   (symbol (lib_id "Device:R_Small") (at 68.58 26.67 270) (unit 1)
     (in_bom yes) (on_board yes) (dnp no)
@@
         (path "/7db990e4-92e1-4f99-b4d2-435bbec1ba83"
           (reference "#PWR021") (unit 1)
+        )
+      )
+    )
+  )
+  (symbol (lib_name "GND_1") (lib_id "power:GND") (at 240.665 104.775 0) (unit 1)
+    (in_bom yes) (on_board yes) (dnp no) (fields_autoplaced)
+    (property "Reference" "#PWR029" (at 240.665 111.125 0)
+      (effects (font (size 1.27 1.27)) hide)
+    )
+    (property "Value" "GND" (at 240.665 109.855 0)
+      (effects (font (size 1.27 1.27)))
+    )
+    (property "Footprint" "" (at 240.665 104.775 0)
+      (effects (font (size 1.27 1.27)) hide)
+    )
+    (property "Datasheet" "" (at 240.665 104.775 0)
+      (effects (font (size 1.27 1.27)) hide)
+    )
+    (pin "1")
+    (instances
+      (project "Ricardo-BlackBoxNEWFinal"
+        (path "/7db990e4-92e1-4f99-b4d2-435bbec1ba83"
+          (reference "#PWR029") (unit 1)
         )
       )
@@
     )
   )
+  (symbol (lib_id "Device:C_Small") (at 240.665 93.345 0) (unit 1)
+    (in_bom yes) (on_board yes) (dnp no) (fields_autoplaced)
+    (property "Reference" "C29" (at 243.205 92.7163 0)
+      (effects (font (size 1.27 1.27)) (justify left))
+    )
+    (property "Value" "0.1uF" (at 243.205 95.2563 0)
+      (effects (font (size 1.27 1.27)) (justify left))
+    )
+    (property "Footprint" "Capacitor_SMD:C_0402_1005Metric" (at 240.665 93.345 0)
+      (effects (font (size 1.27 1.27)) hide)
+    )
+    (property "Datasheet" "~" (at 240.665 93.345 0)
+      (effects (font (size 1.27 1.27)) hide)
+    )
+    (pin "1")
+    (pin "2")
+    (instances
+      (project "Ricardo-BlackBoxNEWFinal"
+        (path "/7db990e4-92e1-4f99-b4d2-435bbec1ba83"
+          (reference "C29") (unit 1)
+        )
+      )
+    )
+  )
   (symbol (lib_id "Connector:TestPoint") (at 229.87 131.445 270) (unit 1)
     (in_bom yes) (on_board yes) (dnp no) (fields_autoplaced)
@@
     )
   )
-  (symbol (lib_id "power:+3.3V") (at 234.315 89.535 0) (unit 1)
+  (symbol (lib_id "power:+3.3V") (at 240.665 88.9 0) (unit 1)
     (in_bom yes) (on_board yes) (dnp no) (fields_autoplaced)
-    (property "Reference" "#PWR0102" (at 234.315 93.345 0)
-      (effects (font (size 1.27 1.27)) hide)
-    )
-    (property "Value" "+3.3V" (at 234.315 84.455 0)
-      (effects (font (size 1.27 1.27)))
-    )
-    (property "Footprint" "" (at 234.315 89.535 0)
-      (effects (font (size 1.27 1.27)) hide)
-    )
-    (property "Datasheet" "" (at 234.315 89.535 0)
+    (property "Reference" "#PWR0102" (at 240.665 92.71 0)
+      (effects (font (size 1.27 1.27)) hide)
+    )
+    (property "Value" "+3.3V" (at 240.665 83.82 0)
+      (effects (font (size 1.27 1.27)))
+    )
+    (property "Footprint" "" (at 240.665 88.9 0)
+      (effects (font (size 1.27 1.27)) hide)
+    )
+    (property "Datasheet" "" (at 240.665 88.9 0)
       (effects (font (size 1.27 1.27)) hide)
     )
@@
       (effects (font (size 1.27 1.27)))
     )
-    (property "Footprint" "Package_DFN_QFN:QFN-56-1EP_7x7mm_P0.4mm_EP5.6x5.6mm" (at 102.87 153.67 0)
+    (property "Footprint" "iclr:QFN40P700X700X90-57N" (at 102.87 153.67 0)
       (effects (font (size 1.27 1.27)) hide)
     )
@@
     )
   )
-  (symbol (lib_id "Device:C_Small") (at 234.315 93.345 0) (unit 1)
+  (symbol (lib_id "Device:C_Small") (at 240.665 102.235 0) (unit 1)
     (in_bom yes) (on_board yes) (dnp no) (fields_autoplaced)
-    (property "Reference" "C28" (at 236.855 92.0812 0)
-      (effects (font (size 1.27 1.27)) (justify left))
-    )
-    (property "Value" "10uF" (at 236.855 94.6212 0)
-      (effects (font (size 1.27 1.27)) (justify left))
-    )
-    (property "Footprint" "Capacitor_SMD:C_0402_1005Metric" (at 234.315 93.345 0)
-      (effects (font (size 1.27 1.27)) hide)
-    )
-    (property "Datasheet" "~" (at 234.315 93.345 0)
-      (effects (font (size 1.27 1.27)) hide)
-    )
+    (property "Reference" "C28" (at 243.205 100.9712 0)
+      (effects (font (size 1.27 1.27)) (justify left))
+    )
+    (property "Value" "10uF" (at 243.205 103.5112 0)
+      (effects (font (size 1.27 1.27)) (justify left))
+    )
+    (property "Footprint" "Capacitor_SMD:C_0402_1005Metric" (at 240.665 102.235 0)
+      (effects (font (size 1.27 1.27)) hide)
+    )
+    (property "Datasheet" "~" (at 240.665 102.235 0)
+      (effects (font (size 1.27 1.27)) hide)
+    )

Commit message: RicardoBlackBox_20_08_2023(2)
Parts:
- removed R7: 3k, Resistor_SMD:R_0402_1005Metric, symbol Device:R_Small
Connections:
- net +3V3: now also C28.1, IC1.8 (VDD)
- net GND: now also C29.2
Other:
- moved on the sheet: C29
Changed lines of the file:
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@@
   (junction (at 53.34 127) (diameter 0) (color 0 0 0 0)
   )
-  (junction (at 58.42 26.67) (diameter 0) (color 0 0 0 0)
+  (junction (at 30.48 191.77) (diameter 0) (color 0 0 0 0)
+  )
+  (junction (at 69.85 142.24) (diameter 0) (color 0 0 0 0)
+  )
+  (junction (at 55.88 127) (diameter 0) (color 0 0 0 0)
+  )
+  (junction (at 245.11 97.155) (diameter 0) (color 0 0 0 0)
+  )
+  (junction (at 63.5 165.1) (diameter 0) (color 0 0 0 0)
+  )
+  (junction (at 59.69 147.32) (diameter 0) (color 0 0 0 0)
+  )
+  (junction (at 62.23 142.24) (diameter 0) (color 0 0 0 0)
+  )
+  (junction (at 34.29 135.89) (diameter 0) (color 0 0 0 0)
+  )
+  (junction (at 20.32 135.89) (diameter 0) (color 0 0 0 0)
+  )
+  (junction (at 45.72 170.18) (diameter 0) (color 0 0 0 0)
   )
   (junction (at 240.665 97.155) (diameter 0) (color 0 0 0 0)
   )
-  (junction (at 30.48 191.77) (diameter 0) (color 0 0 0 0)
-  )
-  (junction (at 69.85 142.24) (diameter 0) (color 0 0 0 0)
-  )
-  (junction (at 55.88 127) (diameter 0) (color 0 0 0 0)
-  )
-  (junction (at 63.5 165.1) (diameter 0) (color 0 0 0 0)
-  )
-  (junction (at 59.69 147.32) (diameter 0) (color 0 0 0 0)
-  )
-  (junction (at 62.23 142.24) (diameter 0) (color 0 0 0 0)
-  )
-  (junction (at 34.29 135.89) (diameter 0) (color 0 0 0 0)
-  )
-  (junction (at 20.32 135.89) (diameter 0) (color 0 0 0 0)
-  )
-  (junction (at 45.72 170.18) (diameter 0) (color 0 0 0 0)
-  )
   (junction (at 29.21 135.89) (diameter 0) (color 0 0 0 0)
   )
@@
   )
   (junction (at 69.85 130.81) (diameter 0) (color 0 0 0 0)
+  )
+  (junction (at 245.11 104.775) (diameter 0) (color 0 0 0 0)
   )
   (junction (at 29.21 140.97) (diameter 0) (color 0 0 0 0)
@@
     (stroke (width 0) (type default))
   )
-  (wire (pts (xy 58.42 26.67) (xy 66.04 26.67))
-    (stroke (width 0) (type default))
-  )
   (wire (pts (xy 16.51 191.77) (xy 20.32 191.77))
     (stroke (width 0) (type default))
@@
     (stroke (width 0) (type default))
   )
+  (wire (pts (xy 245.11 97.155) (xy 249.555 97.155))
+    (stroke (width 0) (type default))
+  )
   (wire (pts (xy 68.58 62.23) (xy 69.85 62.23))
     (stroke (width 0) (type default))
@@
     (stroke (width 0) (type default))
   )
+  (wire (pts (xy 245.11 107.315) (xy 245.11 104.775))
+    (stroke (width 0) (type default))
+  )
   (wire (pts (xy 62.23 142.24) (xy 69.85 142.24))
     (stroke (width 0) (type default))
@@
     (stroke (width 0) (type default))
   )
+  (wire (pts (xy 240.665 97.155) (xy 245.11 97.155))
+    (stroke (width 0) (type default))
+  )
   (wire (pts (xy 156.21 127) (xy 156.21 128.27))
     (stroke (width 0) (type default))
@@
     (stroke (width 0) (type default))
   )
+  (wire (pts (xy 245.11 104.775) (xy 240.665 104.775))
+    (stroke (width 0) (type default))
+  )
   (wire (pts (xy 44.45 135.89) (xy 46.99 135.89))
     (stroke (width 0) (type default))
@@
     (stroke (width 0) (type default))
   )
-  (wire (pts (xy 58.42 21.59) (xy 58.42 26.67))
+  (wire (pts (xy 58.42 21.59) (xy 58.42 40.64))
     (stroke (width 0) (type default))
   )
@@
     (stroke (width 0) (type default))
   )
-  (wire (pts (xy 240.665 97.155) (xy 240.665 95.885))
-    (stroke (width 0) (type default))
-  )
-  (wire (pts (xy 240.665 90.805) (xy 240.665 88.9))
-    (stroke (width 0) (type default))
-  )
   (wire (pts (xy 59.69 67.31) (xy 69.85 67.31))
     (stroke (width 0) (type default))
@@
     (stroke (width 0) (type default))
   )
+  (wire (pts (xy 249.555 97.155) (xy 249.555 99.695))
+    (stroke (width 0) (type default))
+  )
   (wire (pts (xy 230.505 104.775) (xy 235.585 104.775))
     (stroke (width 0) (type default))
   )
-  (wire (pts (xy 58.42 26.67) (xy 58.42 40.64))
-    (stroke (width 0) (type default))
-  )
   (wire (pts (xy 156.21 135.89) (xy 156.21 138.43))
     (stroke (width 0) (type default))
@@
     (stroke (width 0) (type default))
   )
+  (wire (pts (xy 245.11 104.775) (xy 249.555 104.775))
+    (stroke (width 0) (type default))
+  )
   (wire (pts (xy 30.48 191.77) (xy 39.37 191.77))
     (stroke (width 0) (type default))
@@
   )
   (wire (pts (xy 53.34 127) (xy 55.88 127))
-    (stroke (width 0) (type default))
-  )
-  (wire (pts (xy 73.66 26.67) (xy 71.12 26.67))
     (stroke (width 0) (type default))
   )
@@
     )
   )
-  (symbol (lib_id "Device:R_Small") (at 68.58 26.67 270) (unit 1)
-    (in_bom yes) (on_board yes) (dnp no)
-    (property "Reference" "R7" (at 68.58 21.6916 90)
-      (effects (font (size 1.27 1.27)))
-    )
-    (property "Value" "3k" (at 68.58 24.003 90)
-      (effects (font (size 1.27 1.27)))
-    )
-    (property "Footprint" "Resistor_SMD:R_0402_1005Metric" (at 68.58 26.67 0)
-      (effects (font (size 1.27 1.27)) hide)
-    )
-    (property "Datasheet" "~" (at 68.58 26.67 0)
-      (effects (font (size 1.27 1.27)) hide)
-    )
-    (pin "1")
-    (pin "2")
-    (instances
-      (project "Ricardo-BlackBoxNEWFinal"
-        (path "/7db990e4-92e1-4f99-b4d2-435bbec1ba83"
-          (reference "R7") (unit 1)
-        )
-      )
-    )
-  )
   (symbol (lib_id "Connector:TestPoint") (at 29.21 38.1 90) (unit 1)
     (in_bom yes) (on_board yes) (dnp no)
@@
     )
   )
-  (symbol (lib_name "GND_1") (lib_id "power:GND") (at 240.665 104.775 0) (unit 1)
+  (symbol (lib_name "GND_1") (lib_id "power:GND") (at 245.11 107.315 0) (unit 1)
     (in_bom yes) (on_board yes) (dnp no) (fields_autoplaced)
-    (property "Reference" "#PWR029" (at 240.665 111.125 0)
-      (effects (font (size 1.27 1.27)) hide)
-    )
-    (property "Value" "GND" (at 240.665 109.855 0)
-      (effects (font (size 1.27 1.27)))
-    )
-    (property "Footprint" "" (at 240.665 104.775 0)
-      (effects (font (size 1.27 1.27)) hide)
-    )
-    (property "Datasheet" "" (at 240.665 104.775 0)
+    (property "Reference" "#PWR029" (at 245.11 113.665 0)
+      (effects (font (size 1.27 1.27)) hide)
+    )
+    (property "Value" "GND" (at 245.11 112.395 0)
+      (effects (font (size 1.27 1.27)))
+    )
+    (property "Footprint" "" (at 245.11 107.315 0)
+      (effects (font (size 1.27 1.27)) hide)
+    )
+    (property "Datasheet" "" (at 245.11 107.315 0)
       (effects (font (size 1.27 1.27)) hide)
     )
@@
     )
   )
-  (symbol (lib_id "power:+12V") (at 73.66 26.67 0) (unit 1)
-    (in_bom yes) (on_board yes) (dnp no)
-    (property "Reference" "#PWR015" (at 73.66 30.48 0)
-      (effects (font (size 1.27 1.27)) hide)
-    )
-    (property "Value" "+12V" (at 73.66 21.59 0)
-      (effects (font (size 1.27 1.27)))
-    )
-    (property "Footprint" "" (at 73.66 26.67 0)
-      (effects (font (size 1.27 1.27)) hide)
-    )
-    (property "Datasheet" "" (at 73.66 26.67 0)
-      (effects (font (size 1.27 1.27)) hide)
-    )
-    (pin "1")
-    (instances
-      (project "Ricardo-BlackBoxNEWFinal"
-        (path "/7db990e4-92e1-4f99-b4d2-435bbec1ba83"
-          (reference "#PWR015") (unit 1)
-        )
-      )
-    )
-  )
   (symbol (lib_id "Mechanical:MountingHole_Pad") (at 278.13 30.48 0) (unit 1)
     (in_bom yes) (on_board yes) (dnp no)
@@
     )
   )
-  (symbol (lib_id "Device:C_Small") (at 240.665 93.345 0) (unit 1)
+  (symbol (lib_id "Device:C_Small") (at 249.555 102.235 0) (unit 1)
     (in_bom yes) (on_board yes) (dnp no) (fields_autoplaced)
-    (property "Reference" "C29" (at 243.205 92.7163 0)
-      (effects (font (size 1.27 1.27)) (justify left))
-    )
-    (property "Value" "0.1uF" (at 243.205 95.2563 0)
-      (effects (font (size 1.27 1.27)) (justify left))
-    )
-    (property "Footprint" "Capacitor_SMD:C_0402_1005Metric" (at 240.665 93.345 0)
-      (effects (font (size 1.27 1.27)) hide)
-    )
-    (property "Datasheet" "~" (at 240.665 93.345 0)
+    (property "Reference" "C29" (at 252.095 101.6063 0)
+      (effects (font (size 1.27 1.27)) (justify left))
+    )
+    (property "Value" "0.1uF" (at 252.095 104.1463 0)
+      (effects (font (size 1.27 1.27)) (justify left))
+    )
+    (property "Footprint" "Capacitor_SMD:C_0402_1005Metric" (at 249.555 102.235 0)
+      (effects (font (size 1.27 1.27)) hide)
+    )
+    (property "Datasheet" "~" (at 249.555 102.235 0)
       (effects (font (size 1.27 1.27)) hide)
     )
@@
     )
   )
-  (symbol (lib_id "power:+3.3V") (at 240.665 88.9 0) (unit 1)
+  (symbol (lib_id "power:+3.3V") (at 245.11 97.155 0) (unit 1)
     (in_bom yes) (on_board yes) (dnp no) (fields_autoplaced)
-    (property "Reference" "#PWR0102" (at 240.665 92.71 0)
-      (effects (font (size 1.27 1.27)) hide)
-    )
-    (property "Value" "+3.3V" (at 240.665 83.82 0)
-      (effects (font (size 1.27 1.27)))
-    )
-    (property "Footprint" "" (at 240.665 88.9 0)
-      (effects (font (size 1.27 1.27)) hide)
-    )
-    (property "Datasheet" "" (at 240.665 88.9 0)
-      (effects (font (size 1.27 1.27)) hide)
-    )
+    (property "Reference" "#PWR0102" (at 245.11 100.965 0)
+      (effects (font (size 1.27 1.27)) hide)
+    )
+    (property "Value" "+3.3V" (at 245.11 92.075 0)
+      (effects (font (size 1.27 1.27)))
+    )
+    (property "Footprint" "" (at 245.11 97.155 0)
+      (effects (font (size 1.27 1.27)) hide)
+    )
+    (property "Datasheet" "" (at 245.11 97.155 0)
+      (effects (font (size 1.27 1.27)) hide)
+    )

Commit message: RicardoBlackBox_20_08_2023(3)
Connections:
- net MISO: now also U1.41 (GPIO36); no longer U1.40 (GPIO35)
- net MOSI: now also U1.40 (GPIO35); no longer U1.41 (GPIO36)
Changed lines of the file:
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@@
     (effects (font (size 1.27 1.27)) (justify left bottom))
   )
-  (label "MISO" (at 135.89 100.33 0) (fields_autoplaced)
+  (label "MISO" (at 135.89 102.87 0) (fields_autoplaced)
     (effects (font (size 1.27 1.27)) (justify left bottom))
   )
@@
     (effects (font (size 1.27 1.27)) (justify left bottom))
   )
-  (label "MOSI" (at 135.89 102.87 0) (fields_autoplaced)
+  (label "MOSI" (at 135.89 100.33 0) (fields_autoplaced)
     (effects (font (size 1.27 1.27)) (justify left bottom))
   )

Commit message: ordering
Parts:
- 3V3LED1: value 3V3LED -> BLUE_LED
- C12: value 4.2pF -> DNP
- R5: value 47.5 -> DNP
- TXLED1: value TX_LED -> GREEN_LED
- U1: footprint iclr:QFN40P700X700X90-57N -> ICLR:QFN40P700X700X90-57N
Changed lines of the file:
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@@
       (effects (font (size 1.27 1.27)))
     )
-    (property "Value" "TX_LED" (at 25.4 24.4856 0)
+    (property "Value" "GREEN_LED" (at 25.4 24.4856 0)
       (effects (font (size 1.27 1.27)))
     )
@@
       (effects (font (size 1.27 1.27)))
     )
-    (property "Value" "3V3LED" (at 54.61 18.6944 0)
+    (property "Value" "BLUE_LED" (at 54.61 18.6944 0)
       (effects (font (size 1.27 1.27)))
     )
@@
       (effects (font (size 1.27 1.27)) (justify left))
     )
-    (property "Value" "4.2pF" (at 68.58 59.69 90)
+    (property "Value" "DNP" (at 68.58 59.69 90)
       (effects (font (size 1.27 1.27)) (justify left))
     )
@@
       (effects (font (size 1.27 1.27)))
     )
-    (property "Footprint" "iclr:QFN40P700X700X90-57N" (at 102.87 153.67 0)
+    (property "Footprint" "ICLR:QFN40P700X700X90-57N" (at 102.87 153.67 0)
       (effects (font (size 1.27 1.27)) hide)
     )
@@
       (effects (font (size 1.27 1.27)))
     )
-    (property "Value" "47.5" (at 57.15 59.69 90)
-      (effects (font (size 1.27 1.27)))
-    )
+    (property "Value" "DNP" (at 57.15 59.69 90)
+      (effects (font (size 1.27 1.27)))
+    )
